File: modbus_simple_pcb.kicad_sch (KiCad schematic)
At the start: 51 parts, among them J1 L_PinSocket, J10 ADS1115, J11 Screw_Terminal_01x02, J12 Screw_Terminal_01x02, J13 Screw_Terminal_01x02, J14 Screw_Terminal_01x02, J15 KH-2.54FH-1X15P-H8.5, J16 KH-2.54FH-1X15P-H8.5, J17 Screw_Terminal_01x02, J18 Screw_Terminal_01x02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

Commit message: update all resource
Parts:
- R1, R10, R11, R12, R13, R14, R15, R16, R2, R3, R4, R5, R6, R7, R8, R9: value 100 -> 47
Other:
- note added: "GP8403モジュール DFRobot製Gravity GP8403 4個必要です またI2Cアドレスの変更が必須です"
- note added: "J26はオプショナルです 未実装で問題ないです"
- note added: "R1-R16はオプショナルです 0[Ω]としてジャンパしても問題ありません 未実装ではなくジャンパです"
- note added: "R17-R18はオプショナルです 未実装で問題ないです"
- note added: "R70/D8はオプショナルです 未実装で問題ないです"
- note added: "[103216]"
- note removed: "GP8403モジュール DFRobot製Gravity GF8403 4個必要です またI2Cアドレスの変更が必須です"
- moved on the sheet: J21, J22, J23, J24
